File: 7_ESP and Power.kicad_sch (KiCad schematic)
At the start: 44 parts, among them Q1 DMG1013T-7, U1 2, U15 TPS63900DSKR, U16 WAFER-PH2.0-2PWZ, U2 ESP32-C6-MINI-1-N4

Commit message: Fix import2 ERC: pin types, references, and NC pins
- Convert EasyEDA R/C input pins to passive in lib_symbols and symbol library
- Set targeted pin types for ESP32-C6, TYPE-C, ADS1299 NC, TPD4E1B06, TPS62821
- Annotate Short-Symbol jumpers (JP1-6), sheet frames (F1-F2), and #PWR flags
- ERC: 576 violations / 122 errors -> 448 violations / 4 errors
- Net names unchanged; remaining errors are BIASIN/BIASOUT wiring and GND PWR_FLAG
Parts:
- gave numbers to parts that had none: 1
Changed lines of the file:
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@@
 		(in_pos_files yes)
 		(dnp no)
-		(property "Reference" "#PWR?"
+		(property "Reference" "#PWR01"
 			(at 92.71 185.42 0)
 			(hide yes)
@@
 			(project "import2"
 				(path "/06cae45c-d474-473f-93a9-05a684cc4e1b/d7335401-30df-4181-8165-2b729c8075df"
-					(reference "#PWR?")
+					(reference "#PWR02")
 					(unit 1)
 				)
@@
 		(in_pos_files yes)
 		(dnp no)
-		(property "Reference" "#PWR?"
+		(property "Reference" "#PWR03"
 			(at 111.76 127 0)
 			(hide yes)
@@
 			(project "import2"
 				(path "/06cae45c-d474-473f-93a9-05a684cc4e1b/d7335401-30df-4181-8165-2b729c8075df"
-					(reference "#PWR?")
+					(reference "#PWR04")
 					(unit 1)
 				)
@@
 		(in_pos_files yes)
 		(dnp no)
-		(property "Reference" "#PWR?"
+		(property "Reference" "#PWR05"
 			(at 111.76 38.1 0)
 			(hide yes)
@@
 			(project "import2"
 				(path "/06cae45c-d474-473f-93a9-05a684cc4e1b/d7335401-30df-4181-8165-2b729c8075df"
-					(reference "#PWR?")
+					(reference "#PWR06")
 					(unit 1)
 				)
@@
 		(in_pos_files yes)
 		(dnp no)
-		(property "Reference" "#PWR?"
+		(property "Reference" "#PWR07"
 			(at 237.49 66.04 0)
 			(hide yes)
@@
 			(project "import2"
 				(path "/06cae45c-d474-473f-93a9-05a684cc4e1b/d7335401-30df-4181-8165-2b729c8075df"
-					(reference "#PWR?")
+					(reference "#PWR08")
 					(unit 1)
 				)
@@
 		(in_pos_files yes)
 		(dnp no)
-		(property "Reference" "#PWR?"
+		(property "Reference" "#PWR09"
 			(at 284.48 68.58 0)
 			(hide yes)
@@
 			(project "import2"
 				(path "/06cae45c-d474-473f-93a9-05a684cc4e1b/d7335401-30df-4181-8165-2b729c8075df"
-					(reference "#PWR?")
+					(reference "#PWR10")
 					(unit 1)
 				)
@@
 		(in_pos_files yes)
 		(dnp no)
-		(property "Reference" "#PWR?"
+		(property "Reference" "#PWR11"
 			(at 71.12 119.38 0)
 			(hide yes)
@@
 			(project "import2"
 				(path "/06cae45c-d474-473f-93a9-05a684cc4e1b/d7335401-30df-4181-8165-2b729c8075df"
-					(reference "#PWR?")
+					(reference "#PWR12")
 					(unit 1)
 				)
@@
 		(in_pos_files yes)
 		(dnp no)
-		(property "Reference" "#PWR?"
+		(property "Reference" "#PWR13"
 			(at 121.92 127 0)
 			(hide yes)
@@
 			(project "import2"
 				(path "/06cae45c-d474-473f-93a9-05a684cc4e1b/d7335401-30df-4181-8165-2b729c8075df"
-					(reference "#PWR?")
+					(reference "#PWR14")
 					(unit 1)
 				)
@@
 		(in_pos_files yes)
 		(dnp no)
-		(property "Reference" "#PWR?"
+		(property "Reference" "#PWR15"
 			(at 304.8 166.37 0)
 			(hide yes)
@@
 			(project "import2"
 				(path "/06cae45c-d474-473f-93a9-05a684cc4e1b/d7335401-30df-4181-8165-2b729c8075df"
-					(reference "#PWR?")
+					(reference "#PWR16")
 					(unit 1)
 				)
@@
 		(in_pos_files yes)
 		(dnp no)
-		(property "Reference" "?"
+		(property "Reference" "JP1"
 			(at 336.042 228.727 0)
 			(show_name no)
@@
 			(project "import2"
 				(path "/06cae45c-d474-473f-93a9-05a684cc4e1b/d7335401-30df-4181-8165-2b729c8075df"
-					(reference "?")
+					(reference "JP1")
 					(unit 0)
 				)
@@
 		(in_pos_files yes)
 		(dnp no)
-		(property "Reference" "#PWR?"
+		(property "Reference" "#PWR17"
 			(at 156.21 31.75 0)
 			(hide yes)
@@
 			(project "import2"
 				(path "/06cae45c-d474-473f-93a9-05a684cc4e1b/d7335401-30df-4181-8165-2b729c8075df"
-					(reference "#PWR?")
+					(reference "#PWR18")
 					(unit 1)
 				)
@@
 		(in_pos_files yes)
 		(dnp no)
-		(property "Reference" "#PWR?"
+		(property "Reference" "#PWR19"
 			(at 78.74 93.98 0)
 			(hide yes)
@@
 			(project "import2"
 				(path "/06cae45c-d474-473f-93a9-05a684cc4e1b/d7335401-30df-4181-8165-2b729c8075df"
-					(reference "#PWR?")
+					(reference "#PWR20")
 					(unit 1)
 				)
@@
 		(in_pos_files yes)
 		(dnp no)
-		(property "Reference" "#PWR?"
+		(property "Reference" "#PWR21"
 			(at 93.98 218.44 0)
 			(hide yes)
@@
 			(project "import2"
 				(path "/06cae45c-d474-473f-93a9-05a684cc4e1b/d7335401-30df-4181-8165-2b729c8075df"
-					(reference "#PWR?")
+					(reference "#PWR22")
 					(unit 1)
 				)
@@
 		(in_pos_files yes)
 		(dnp no)
-		(property "Reference" "#PWR?"
+		(property "Reference" "#PWR23"
 			(at 304.8 29.21 0)
 			(hide yes)
@@
 			(project "import2"
 				(path "/06cae45c-d474-473f-93a9-05a684cc4e1b/d7335401-30df-4181-8165-2b729c8075df"
-					(reference "#PWR?")
+					(reference "#PWR24")
 					(unit 1)
 				)
@@
 		(in_pos_files yes)
 		(dnp no)
-		(property "Reference" "#PWR?"
+		(property "Reference" "#PWR25"
 			(at 43.18 190.5 0)
 			(hide yes)
@@
 			(project "import2"
 				(path "/06cae45c-d474-473f-93a9-05a684cc4e1b/d7335401-30df-4181-8165-2b729c8075df"
-					(reference "#PWR?")
+					(reference "#PWR26")
 					(unit 1)
 				)
@@
 		(in_pos_files yes)
 		(dnp no)
-		(property "Reference" "#PWR?"
+		(property "Reference" "#PWR27"
 			(at 110.49 55.88 0)
 			(hide yes)
@@
 			(project "import2"
 				(path "/06cae45c-d474-473f-93a9-05a684cc4e1b/d7335401-30df-4181-8165-2b729c8075df"
-					(reference "#PWR?")
+					(reference "#PWR28")
 					(unit 1)
 				)
@@
 		(in_pos_files yes)
 		(dnp no)
-		(property "Reference" "#PWR?"
+		(property "Reference" "#PWR29"
 			(at 54.61 218.44 0)
 			(hide yes)
@@
 			(project "import2"
 				(path "/06cae45c-d474-473f-93a9-05a684cc4e1b/d7335401-30df-4181-8165-2b729c8075df"
-					(reference "#PWR?")
+					(reference "#PWR30")
 					(unit 1)
 				)
@@
 		(in_pos_files yes)
 		(dnp no)
-		(property "Reference" "#PWR?"
+		(property "Reference" "#PWR31"
 			(at 71.12 106.68 0)
 			(hide yes)
@@
 			(project "import2"
 				(path "/06cae45c-d474-473f-93a9-05a684cc4e1b/d7335401-30df-4181-8165-2b729c8075df"
-					(reference "#PWR?")
+					(reference "#PWR32")
 					(unit 1)
 				)
@@
 		(in_pos_files yes)
 		(dnp no)
-		(property "Reference" "#PWR?"
+		(property "Reference" "#PWR33"
 			(at 31.75 68.58 0)
 			(hide yes)
@@
 			(project "import2"
 				(path "/06cae45c-d474-473f-93a9-05a684cc4e1b/d7335401-30df-4181-8165-2b729c8075df"
-					(reference "#PWR?")
+					(reference "#PWR34")
 					(unit 1)
 				)
@@
 		(in_pos_files yes)
 		(dnp no)
-		(property "Reference" "#PWR?"
+		(property "Reference" "#PWR35"
 			(at 273.05 123.19 0)
 			(hide yes)
@@
 			(project "import2"
 				(path "/06cae45c-d474-473f-93a9-05a684cc4e1b/d7335401-30df-4181-8165-2b729c8075df"
-					(reference "#PWR?")
+					(reference "#PWR36")
 					(unit 1)
 				)
@@
 		(in_pos_files yes)
 		(dnp no)
-		(property "Reference" "#PWR?"
+		(property "Reference" "#PWR37"
 			(at 43.18 119.38 0)
 			(hide yes)
@@
 			(project "import2"
 				(path "/06cae45c-d474-473f-93a9-05a684cc4e1b/d7335401-30df-4181-8165-2b729c8075df"
-					(reference "#PWR?")
+					(reference "#PWR38")
 					(unit 1)
 				)
@@
 		(in_pos_files yes)
 		(dnp no)
-		(property "Reference" "#PWR?"
+		(property "Reference" "#PWR39"
 			(at 92.71 195.58 0)
 			(hide yes)
@@
 			(project "import2"
 				(path "/06cae45c-d474-473f-93a9-05a684cc4e1b/d7335401-30df-4181-8165-2b729c8075df"
-					(reference "#PWR?")
+					(reference "#PWR40")
 					(unit 1)
 				)
@@
 		(in_pos_files yes)
 		(dnp no)
-		(property "Reference" "#PWR?"
+		(property "Reference" "#PWR41"
 			(at 124.46 114.3 0)
 			(hide yes)
@@
 			(project "import2"
 				(path "/06cae45c-d474-473f-93a9-05a684cc4e1b/d7335401-30df-4181-8165-2b729c8075df"
-					(reference "#PWR?")
+					(reference "#PWR42")
 					(unit 1)
 				)
@@
 		(in_pos_files yes)
 		(dnp no)
-		(property "Reference" "#PWR?"
+		(property "Reference" "#PWR43"
 			(at 90.17 139.7 0)
 			(hide yes)
@@
 			(project "import2"
 				(path "/06cae45c-d474-473f-93a9-05a684cc4e1b/d7335401-30df-4181-8165-2b729c8075df"
-					(reference "#PWR?")
+					(reference "#PWR44")
 					(unit 1)
 				)
@@
 		(in_pos_files yes)
 		(dnp no)
-		(property "Reference" "#PWR?"
+		(property "Reference" "#PWR45"
 			(at 100.33 173.99 0)
 			(hide yes)
@@
 			(project "import2"
 				(path "/06cae45c-d474-473f-93a9-05a684cc4e1b/d7335401-30df-4181-8165-2b729c8075df"
-					(reference "#PWR?")
+					(reference "#PWR46")
 					(unit 1)
 				)

Commit message: Fix ERC
Parts:
- removed JP1: (no value), ProPrj_BCI-easyedapro:, symbol ProPrj_BCI-easyedapro:Short-Symbol-Auto
- P1: footprint ProPrj_BCI-easyedapro: -> normalized-easyedapro:SOT-23-6_L2.9-W1.6-P0.95-LS2.8-BL
- renumbered C_adc to C_adc1
Connections:
- net 3V3: now also U1.6
- net 5V: no longer U1.6
- net B: now also U2.24 (IO18)
- net PWDN: no longer U2.19 (IO14)
- net 5V_PMOD renamed 3V3_PMOD
- net IO3 renamed INT
- new net SCLK: U2.19 (IO14)
- no-connect marks 9 -> 8

Commit message: Add boot and reset buttonss
Parts:
- added C224: 1uF, normalized-easyedapro:C0603, symbol ProPrj_BCI-easyedapro:GRM219R61A106KE44D
- added RBOOT, RPWDN: 10kΩ, ProPrj_BCI-easyedapro:R0402, symbol ProPrj_BCI-easyedapro:0402WGF2001TCE
- added SW1, SW2: PTS810SJM250SMTRLFS, jlcpcb:KEY-SMD_4P-L4.2-W3.2-P2.20-LS4.6, symbol jlcpcb:PTS810SJM250SMTRLFS
Connections:
- net 3V3_MCU: now also RBOOT.1, RPWDN.1
- net GND: now also C224.2, SW1.2, SW2.2
- net HOST_INT: now also U2.25 (IO19); no longer U2.23 (IO9)
- net PWDN: now also RPWDN.2
- net RST: now reaches R1.2, U2.8 (EN)
- net RST: now also C224.1, SW1.4
- new net BOOT: RBOOT.2, SW2.4, U2.23 (IO9)
- no-connect marks 8 -> 11

Commit message: PCB update. DRC <300
Parts:
- renumbered RBOOT to RBOOT1, RPWDN to RPWDN1
Changed lines of the file:
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@@
 		(in_pos_files yes)
 		(dnp no)
-		(property "Reference" "RBOOT"
+		(property "Reference" "RBOOT1"
 			(at 181.61 176.53 0)
 			(show_name no)
@@
 			(project "import2"
 				(path "/06cae45c-d474-473f-93a9-05a684cc4e1b/d7335401-30df-4181-8165-2b729c8075df"
-					(reference "RBOOT")
+					(reference "RBOOT1")
 					(unit 1)
 				)
@@
 		(in_pos_files yes)
 		(dnp no)
-		(property "Reference" "RPWDN"
+		(property "Reference" "RPWDN1"
 			(at 161.29 153.67 0)
 			(show_name no)
@@
 			(project "import2"
 				(path "/06cae45c-d474-473f-93a9-05a684cc4e1b/d7335401-30df-4181-8165-2b729c8075df"
-					(reference "RPWDN")
+					(reference "RPWDN1")
 					(unit 1)
 				)
