File: import2.kicad_pcb (KiCad board)
At the start: 4 copper layers, 59.3 x 46.4 mm, 165 parts, among them Q1 DMG1013T-7, SW1 PTS810SJM250SMTRLFS, SW2 PTS810SJM250SMTRLFS, U1 2, U15 TPS63900DSKR, U16 WAFER-PH2.0-2PWZ, U2 ESP32-C6-MINI-1-N4, U3 SLW-913535-2A-SMT

Commit message: No errors. Only silk warnings
Parts:
- moved C29 3.36 mm to (161.1, 94.2), turned to 90 degrees
- moved C28 3.18 mm to (159.5, 94.2), turned to 90 degrees
- moved R_adc1 2.68 mm to (160.7, 99.2), turned to -90 degrees
- moved C41 2.50 mm to (160.3, 113.2), turned to 180 degrees
- moved Rb1 2.46 mm to (163.1, 119.3)
- moved C42 2.11 mm to (160.3, 114.8), turned to 180 degrees
- moved C222 1.78 mm to (159.9, 91.2)
- moved C223 1.75 mm to (161.4, 91.2)
- moved C37 1.67 mm to (155.3, 109.8), turned to -90 degrees
- moved RL2 1.26 mm to (170.8, 104.4)
- moved C234 1.05 mm to (166.6, 121.9)
- moved LED2 0.96 mm to (172.0, 104.5)
- moved RBIAS1 0.87 mm to (149.3, 88.8)
- moved R1 0.85 mm to (161.2, 96.4), turned to 0 degrees
- moved F1 0.77 mm to (168.8, 113.8), turned to 0 degrees
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Routing:
- net GND: track 75.5 -> 32.6 mm, vias 35 -> 32
- net (no net): track 22.6 -> 0.00 mm, vias 2 -> 0
- net MOSI: track 47.1 -> 34.3 mm, vias 5 -> 4
- net 5V_ADC: track 126.8 -> 139.1 mm
- net BAT+: track 6.87 -> 0.07 mm
- net VSYS: track 24.6 -> 18.6 mm, vias 2 -> 1
- net VIN: track 58.2 -> 63.3 mm, vias 7 -> 6
- net 3V3_MCU: track 48.6 -> 53.1 mm
- net 3V3_ADC: track 59.7 -> 63.7 mm
- net CSEL2: track 26.9 -> 23.1 mm
- net DN: track 25.4 -> 22.1 mm, vias 3 -> 2
- net MISO: track 10.9 -> 8.14 mm
- net SLAVE_DOUT: track 24.3 -> 21.8 mm
- net PINSRB2: track 32.8 -> 30.4 mm
- net AVSS: track 32.5 -> 30.4 mm, vias 15 -> 31
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- added copper zone on F.Cu, net 3V3_MCU
- added copper zone on F.Cu, net Net-(U15-LX1)
- added copper zone on F.Cu, net Net-(U15-LX2)
- removed copper zone on B.Cu, net 3V3
- removed copper zone on In1.Cu, net 3V3
- removed copper zone on In2.Cu, net 3V3
- removed copper zone on B.Cu, net 5V
- removed copper zone on In1.Cu, net 5V
- removed copper zone on In2.Cu, net 5V
- removed copper zone on B.Cu, net USB_5V_IN
- removed copper zone on In1.Cu, net USB_5V_IN
- removed copper zone on In2.Cu, net USB_5V_IN
- removed copper zone on B.Cu, net VIN
Other:
- outline, holes or cut-outs redrawn
