File: _restore_backup_2026-08-23T15-10-23-191/import2.kicad_pcb (KiCad board)
At the start: 4 copper layers, 59.3 x 46.4 mm, 165 parts, among them Q1 DMG1013T-7, SW1 PTS810SJM250SMTRLFS, SW2 PTS810SJM250SMTRLFS, U1 2, U15 TPS63900DSKR, U16 WAFER-PH2.0-2PWZ, U2 ESP32-C6-MINI-1-N4, U3 SLW-913535-2A-SMT

Commit message: Add buttons. Rework PSU placement. No missed connections. 220 errors
Parts:
- moved Rb1 1.69 mm to (163.5, 120.0), turned to 0 degrees
- moved C233 1.63 mm to (174.7, 106.8), turned to -90 degrees
- moved Rb3 0.87 mm to (174.7, 103.9), turned to -90 degrees
- moved Rb2 0.66 mm to (164.8, 119.5)
- moved Rb4 0.62 mm to (175.6, 103.9)
- moved C227 0.54 mm to (164.9, 117.6)
- moved Rb6 0.47 mm to (177.3, 102.9)
- moved Rb5 0.43 mm to (176.4, 103.9)
- moved L2 0.27 mm to (176.6, 109.3)
- moved NT5 0.25 mm to (158.8, 103.4)
- moved Rb7 0.08 mm to (177.8, 104.1)
Routing:
- net (no net): track 22.6 -> 48.7 mm, vias 2 -> 5
- net BIAS_DRV: track 7.21 -> 32.4 mm, vias 1 -> 4
- net GND: track 75.5 -> 52.2 mm, vias 35 -> 15
- net VSYS: track 24.6 -> 6.00 mm
- net RESET: track 37.3 -> 25.3 mm
- net Net-(ADC1-BIASIN): track 5.08 -> 0.00 mm
- net BIASINV: track 28.6 -> 24.9 mm
- net VIN: track 58.2 -> 54.7 mm, vias 7 -> 6
- net INT: track 6.48 -> 4.33 mm, vias 2 -> 1
- net 3V3_MCU: track 48.6 -> 46.5 mm
- net USB_5V: track 17.7 -> 16.1 mm
- net Net-(ADC1-VCAP3): track 3.09 -> 1.49 mm, vias 0 -> 2
- net 5V_ADC: track 126.8 -> 125.5 mm
- net 5V: track 39.2 -> 40.3 mm
- net /ESP and Power/HOST_UART_RTS: track 32.9 -> 31.9 mm
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- added copper zone on In1.Cu, net VIN
- added copper zone on In2.Cu, net VIN
Other:
- outline, holes or cut-outs redrawn
